File: juggling_machine_pcb/_autosave-juggling_machine_pcb.kicad_pcb (KiCad board)
At the start: 2 copper layers, 97 x 95 mm, 16 parts, among them J1 Conn_01x08, J10 Screw_Terminal_01x04, J11 Screw_Terminal_01x04, J2 Conn_01x08, J3 Conn_01x08, J4 Conn_01x08, J5 servo 1, J6 servo 2, J7 24v input, J8 5v input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

Commit message: added new BOM, plus updated pcb
Routing:
- net +24V: track 109.6 -> 99.3 mm
- net MOSI: track 151.7 -> 144.9 mm
- net +5V: track 197.2 -> 191.5 mm, vias 6 -> 5
- net SCK: track 163.2 -> 160.0 mm, vias 1 -> 3
- net Net-(A1-GPIO22): track 88.5 -> 85.7 mm
- net Net-(J7-Pin_1): track 101.9 -> 100.3 mm, vias 1 -> 0
- net Net-(A1-GPIO15): track 108.6 -> 110.0 mm
- net Net-(D2-K): track 45.9 -> 44.9 mm
- net Net-(D1-A): track 45.6 -> 46.2 mm
- net Net-(J10-Pin_1): vias 2 -> 1
- net GND: vias 0 -> 1
