File: juggling_machine_pcb/juggling_machine_pcb.kicad_pcb (KiCad board)
At the start: 2 copper layers, 97 x 95 mm, 16 parts, among them J1 Conn_01x08, J10 Screw_Terminal_01x04, J11 Screw_Terminal_01x04, J2 Conn_01x08, J3 Conn_01x08, J4 Conn_01x08, J5 servo 1, J6 servo 2, J7 24v input, J8 5v input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

Commit message: added new BOM, plus updated pcb
Routing:
- net Net-(J7-Pin_1): track 101.9 -> 77.6 mm, vias 1 -> 0
- net MOSI: track 151.7 -> 144.8 mm
- net +5V: vias 6 -> 5
- net Net-(J10-Pin_1): vias 2 -> 1
Changed lines of the file:
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@@
 	)
 	(segment
-		(start 54.5 59.275793)
-		(end 54.5 74.875)
+		(start 86.9465 61.630929)
+		(end 86.9465 73.6715)
 		(width 0.2)
 		(layer "B.Cu")
@@
 	)
 	(segment
-		(start 88.75 75.475)
-		(end 85.727 72.452)
-		(width 0.2)
-		(layer "B.Cu")
-		(net 11)
-	)
-	(segment
-		(start 82.288571 56.973)
-		(end 56.802793 56.973)
-		(width 0.2)
-		(layer "B.Cu")
-		(net 11)
-	)
-	(segment
-		(start 85.727 60.411429)
-		(end 82.288571 56.973)
+		(start 86.9465 73.6715)
+		(end 88.75 75.475)
 		(width 0.2)
 		(layer "B.Cu")
@@
 	)
 	(segment
-		(start 54.5 75.175)
-		(end 54.5 83.875)
-		(width 0.2)
-		(layer "B.Cu")
-		(net 11)
-	)
-	(segment
 		(start 94.768081 88.374)
 		(end 90.777081 92.365)
@@
 	)
 	(segment
+		(start 54.7 84.275)
+		(end 54.7 70.657322)
+		(width 0.2)
+		(layer "B.Cu")
+		(net 11)
+	)
+	(segment
+		(start 54.7 70.657322)
+		(end 68.084322 57.273)
+		(width 0.2)
+		(layer "B.Cu")
+		(net 11)
+	)
+	(segment
 		(start 109.425 91.533)
 		(end 106.266 88.374)
@@
 	)
 	(segment
-		(start 54.5 74.875)
-		(end 54.5 75.175)
+		(start 82.588571 57.273)
+		(end 86.9465 61.630929)
 		(width 0.2)
 		(layer "B.Cu")
@@
 	)
 	(segment
-		(start 56.802793 56.973)
-		(end 54.5 59.275793)
-		(width 0.2)
-		(layer "B.Cu")
-		(net 11)
-	)
-	(segment
 		(start 109.425 95.45)
 		(end 109.425 91.533)
@@
 	)
 	(segment
-		(start 85.727 72.452)
-		(end 85.727 60.411429)
-		(width 0.2)
-		(layer "B.Cu")
-		(net 11)
-	)
-	(segment
-		(start 54.5 83.875)
-		(end 54.5 84.075)
+		(start 68.084322 57.273)
+		(end 82.588571 57.273)
 		(width 0.2)
 		(layer "B.Cu")
@@
 	)
 	(segment
-		(start 76.0025 35.9725)
-		(end 74.775 37.2)
-		(width 0.5)
-		(layer "F.Cu")
+		(start 72.774 35.774)
+		(end 72.774 33.06258)
+		(width 0.2)
+		(layer "B.Cu")
 		(net 32)
 	)
 	(segment
-		(start 79.675 33.85)
-		(end 77.5525 35.9725)
-		(width 0.5)
-		(layer "F.Cu")
+		(start 77.774 31.949)
+		(end 79.675 33.85)
+		(width 0.2)
+		(layer "B.Cu")
 		(net 32)
 	)
 	(segment
-		(start 77.5525 35.9725)
-		(end 76.0025 35.9725)
-		(width 0.5)
-		(layer "F.Cu")
+		(start 133.125 48.2)
+		(end 85.2 48.2)
+		(width 0.5)
+		(layer "B.Cu")
 		(net 32)
 	)
 	(segment
-		(start 74.775 39.175)
-		(end 72.5 41.45)
-		(width 0.5)
-		(layer "F.Cu")
+		(start 85.2 48.2)
+		(end 77.9 40.9)
+		(width 0.5)
+		(layer "B.Cu")
 		(net 32)
 	)
 	(segment
-		(start 74.775 37.2)
-		(end 74.775 39.175)
-		(width 0.5)
-		(layer "F.Cu")
+		(start 77.9 40.9)
+		(end 72.774 35.774)
+		(width 0.2)
+		(layer "B.Cu")
 		(net 32)
 	)
 	(segment
-		(start 72.5 41.45)
-		(end 68.625 41.45)
-		(width 0.5)
-		(layer "F.Cu")
+		(start 134 47.325)
+		(end 133.125 48.2)
+		(width 0.5)
+		(layer "B.Cu")
 		(net 32)
 	)
 	(segment
-		(start 68.625 41.45)
-		(end 68.275 41.1)
-		(width 0.5)
-		(layer "F.Cu")
+		(start 72.774 33.06258)
+		(end 73.88758 31.949)
+		(width 0.2)
+		(layer "B.Cu")
 		(net 32)
 	)
-	(via
-		(at 68.275 41.1)
-		(size 0.6)
-		(drill 0.3)
-		(layers "F.Cu" "B.Cu")
-		(net 32)
-	)
-	(segment
-		(start 133.125 48.2)
-		(end 134 47.325)
-		(width 0.5)
-		(layer "B.Cu")
-		(net 32)
-	)
-	(segment
-		(start 61.65 47.225)
-		(end 61.65 44.525)
-		(width 0.5)
-		(layer "B.Cu")
-		(net 32)
-	)
-	(segment
-		(start 65.075 41.1)
-		(end 68.275 41.1)
-		(width 0.5)
-		(layer "B.Cu")
-		(net 32)
-	)
-	(segment
-		(start 65.275 50.85)
-		(end 62.7 48.275)
-		(width 0.5)
-		(layer "B.Cu")
-		(net 32)
-	)
-	(segment
-		(start 61.65 44.525)
-		(end 65.075 41.1)
-		(width 0.5)
-		(layer "B.Cu")
-		(net 32)
-	)
-	(segment
-		(start 82.55 50.85)
-		(end 85.2 48.2)
-		(width 0.5)
-		(layer "B.Cu")
-		(net 32)
-	)
-	(segment
-		(start 82.55 50.85)
-		(end 65.275 50.85)
-		(width 0.5)
-		(layer "B.Cu")
-		(net 32)
-	)
-	(segment
-		(start 85.2 48.2)
-		(end 133.125 48.2)
-		(width 0.5)
-		(layer "B.Cu")
-		(net 32)
-	)
-	(segment
-		(start 62.7 48.275)
-		(end 61.65 47.225)
-		(width 0.5)
+	(segment
+		(start 73.88758 31.949)
+		(end 77.774 31.949)
+		(width 0.2)
 		(layer "B.Cu")
 		(net 32)
@@
 		(net 37)
 	)
-	(segment
-		(start 113 103.09)
-		(end 113 104)
-		(width 0.2)
-		(layer "F.Cu")
-		(net 37)
-	)
-	(segment
-		(start 104.815 94.905)
-		(end 113 103.09)
-		(width 0.2)
-		(layer "F.Cu")
-		(net 37)
-	)
-	(via
-		(at 113 104)
-		(size 0.6)
-		(drill 0.3)
-		(layers "F.Cu" "B.Cu")
-		(net 37)
-	)
 	(via
 		(at 117 108)
@@
 	)
 	(segment
+		(start 113 103.09)
+		(end 104.815 94.905)
+		(width 0.2)
+		(layer "B.Cu")
+		(net 37)
+	)
+	(segment
+		(start 113 104)
+		(end 113 103.09)
+		(width 0.2)
+		(layer "B.Cu")
+		(net 37)
+	)
+	(segment
 		(start 102.305 28.945)
 		(end 101.4 29.85)
@@
 	)
 	(segment
-		(start 114.24 58.315)
-		(end 116.15 60.225)
-		(width 0.2)
-		(layer "F.Cu")
-		(net 41)
-	)
-	(segment
 		(start 62 114)
 		(end 61.891 114.109)
@@
 	)
 	(segment
-		(start 114.24 56.375)
-		(end 114.24 58.315)
-		(width 0.2)
-		(layer "F.Cu")
-		(net 41)
-	)
-	(segment
 		(start 108.275 31.485)
 		(end 114.085 31.485)
@@
 	)
 	(via
-		(at 116.15 60.225)
-		(size 0.6)
-		(drill 0.3)
-		(layers "F.Cu" "B.Cu")
-		(net 41)
-	)
-	(via
 		(at 87.25 87.875)
 		(size 0.6)
@@
 	)
 	(segment
-		(start 118.975 60.225)
-		(end 121.375 62.625)
+		(start 121.775 65.85)
+		(end 121.775 63.025)
+		(width 0.2)
+		(layer "B.Cu")
+		(net 41)
+	)
+	(segment
+		(start 100 83.825)
+		(end 103.8 83.825)
 		(width 0.2)
 		(layer "B.Cu")
@@
 	)
 	(segment
-		(start 116.15 60.225)
+		(start 121.775 63.025)
 		(end 118.975 60.225)
-		(width 0.2)
-		(layer "B.Cu")
-		(net 41)
-	)
-	(segment
-		(start 121.775 65.85)
-		(end 103.8 83.825)
 		(width 0.2)
 		(layer "B.Cu")
@@
 	)
 	(segment
-		(start 121.775 63.025)
+		(start 103.8 83.825)
 		(end 121.775 65.85)
 		(width 0.2)
@@
 	)
 	(segment
-		(start 121.375 62.625)
-		(end 121.775 63.025)
-		(width 0.2)
-		(layer "B.Cu")
-		(net 41)
-	)
-	(segment
-		(start 103.8 83.825)
-		(end 100 83.825)
+		(start 118.975 60.225)
+		(end 116.15 60.225)
+		(width 0.2)
+		(layer "B.Cu")
+		(net 41)
+	)
+	(segment
+		(start 116.15 60.225)
+		(end 114.24 58.315)
 		(width 0.2)
 		(layer "B.Cu")
@@
 		(width 0.2)
 		(layer "B.Cu")
+		(net 41)
+	)
+	(segment
+		(start 114.24 58.315)
+		(end 114.24 56.375)
+		(width 0.2)
+		(layer "B.Cu")

Commit message: latest changes
Routing:
- net Net-(J7-Pin_1): track 77.6 -> 100.3 mm
- net +24V: track 109.6 -> 99.3 mm
- net +5V: track 197.2 -> 191.5 mm
- net SCK: track 163.2 -> 160.0 mm, vias 1 -> 3
- net Net-(A1-GPIO22): track 88.5 -> 85.7 mm
- net Net-(A1-GPIO15): track 108.6 -> 110.0 mm
- net Net-(D2-K): track 45.9 -> 44.9 mm
- net Net-(D1-A): track 45.6 -> 46.2 mm
- net GND: vias 0 -> 1
